File: ioboard.kicad_pcb (KiCad board)
At the start: 2 copper layers, 48.3 x 108 mm, 42 parts, among them U3 TL431DBZ

Commit message: asd
Parts:
- R14: value 10k -> DNP
- R15: value 5k6 -> DNP
- R2: value 3.3M -> 2.2M
- moved U3 1.06 mm to (135.3, 62.7), turned to 0 degrees
Routing:
- net /MULTI-IN: track 59.0 -> 93.6 mm
- net Net-(U1-C): track 0.00 -> 4.59 mm
- net GND: track 6.98 -> 10.5 mm
Changed lines of the file:
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@@
 			)
 		)
-		(property "Value" "3.3M"
+		(property "Value" "2.2M"
 			(at 0 -1.65 90)
 			(layer "B.Fab")
@@
 	(footprint "Package_TO_SOT_SMD:SOT-23"
 		(layer "B.Cu")
-		(at 134.23 62.712 180)
+		(at 135.2925 62.712)
 		(descr "SOT, 3 Pin (JEDEC TO-236 Var AB https://www.jedec.org/document_search?search_api_views_fulltext=TO-236), generated with kicad-footprint-generator ipc_gullwing_generator.py")
 		(tags "SOT TO_SOT_SMD")
 		(property "Reference" "U3"
-			(at 0 2.4 0)
+			(at 0 2.4 180)
 			(layer "B.SilkS")
 			(effects
@@
 		)
 		(property "Value" "TL431DBZ"
-			(at 0 -2.4 0)
+			(at 0 -2.4 180)
 			(layer "B.Fab")
 			(effects
@@
 		)
 		(property "Footprint" "Package_TO_SOT_SMD:SOT-23"
-			(at 0 0 0)
+			(at 0 0 180)
 			(layer "B.Fab")
 			(hide yes)
@@
 		)
 		(property "Datasheet" "http://www.ti.com/lit/ds/symlink/tl431.pdf"
-			(at 0 0 0)
+			(at 0 0 180)
 			(layer "B.Fab")
 			(hide yes)
@@
 		)
 		(property "Description" "Shunt Regulator, SOT-23"
-			(at 0 0 0)
+			(at 0 0 180)
 			(layer "B.Fab")
 			(hide yes)
@@
 		(attr smd)
 		(fp_line
-			(start 0.65 1.56)
-			(end 0 1.56)
+			(start -0.65 -1.56)
+			(end 0 -1.56)
 			(stroke
 				(width 0.12)
@@
 		)
 		(fp_line
-			(start 0.65 -1.56)
-			(end 0 -1.56)
+			(start -0.65 1.56)
+			(end 0 1.56)
 			(stroke
 				(width 0.12)
@@
 		)
 		(fp_line
-			(start -0.65 1.56)
-			(end 0 1.56)
+			(start 0.65 -1.56)
+			(end 0 -1.56)
 			(stroke
 				(width 0.12)
@@
 		)
 		(fp_line
-			(start -0.65 -1.56)
-			(end 0 -1.56)
+			(start 0.65 1.56)
+			(end 0 1.56)
 			(stroke
 				(width 0.12)
@@
 		)
 		(fp_line
-			(start 1.92 1.7)
-			(end 1.92 -1.7)
+			(start -1.92 -1.7)
+			(end -1.92 1.7)
 			(stroke
 				(width 0.05)
@@
 		)
 		(fp_line
-			(start 1.92 -1.7)
-			(end -1.92 -1.7)
+			(start -1.92 1.7)
+			(end 1.92 1.7)
 			(stroke
 				(width 0.05)
@@
 		)
 		(fp_line
-			(start -1.92 1.7)
-			(end 1.92 1.7)
+			(start 1.92 -1.7)
+			(end -1.92 -1.7)
 			(stroke
 				(width 0.05)
@@
 		)
 		(fp_line
-			(start -1.92 -1.7)
-			(end -1.92 1.7)
+			(start 1.92 1.7)
+			(end 1.92 -1.7)
 			(stroke
 				(width 0.05)
@@
 		)
 		(fp_line
-			(start 0.65 1.45)
-			(end -0.325 1.45)
+			(start -0.65 -1.45)
+			(end 0.65 -1.45)
 			(stroke
 				(width 0.1)
@@
 		)
 		(fp_line
-			(start 0.65 -1.45)
-			(end 0.65 1.45)
+			(start -0.65 1.125)
+			(end -0.65 -1.45)
 			(stroke
 				(width 0.1)
@@
 		)
 		(fp_line
-			(start -0.65 1.125)
-			(end -0.65 -1.45)
+			(start 0.65 -1.45)
+			(end 0.65 1.45)
 			(stroke
 				(width 0.1)
@@
 		)
 		(fp_line
-			(start -0.65 -1.45)
-			(end 0.65 -1.45)
+			(start 0.65 1.45)
+			(end -0.325 1.45)
 			(stroke
 				(width 0.1)
@@
 		)
 		(fp_text user "${REFERENCE}"
-			(at 0 0 0)
+			(at 0 0 180)
 			(layer "B.Fab")
 			(effects
@@
 		)
 		(pad "1" smd roundrect
-			(at -0.9375 0.95 180)
+			(at -0.9375 -0.95)
 			(size 1.475 0.6)
 			(layers "B.Cu" "B.Paste" "B.Mask")
@@
 		)
 		(pad "2" smd roundrect
-			(at -0.9375 -0.95 180)
+			(at -0.9375 0.95)
 			(size 1.475 0.6)
 			(layers "B.Cu" "B.Paste" "B.Mask")
@@
 		)
 		(pad "3" smd roundrect
-			(at 0.9375 0 180)
+			(at 0.9375 0)
 			(size 1.475 0.6)
 			(layers "B.Cu" "B.Paste" "B.Mask")
@@
 			)
 		)
-		(property "Value" "10k"
+		(property "Value" "DNP"
 			(at 0 -1.65 90)
 			(layer "B.Fab")
@@
 			)
 		)
-		(property "Value" "5k6"
+		(property "Value" "DNP"
 			(at 0 -1.65 0)
 			(layer "B.Fab")
@@
 	)
 	(segment
+		(start 136.23 62.712)
+		(end 133.538 62.712)
+		(width 0.25)
+		(layer "B.Cu")
+		(net 1)
+	)
+	(segment
+		(start 133.538 62.712)
+		(end 132.73 63.52)
+		(width 0.25)
+		(layer "B.Cu")
+		(net 1)
+	)
+	(segment
+		(start 132.73 63.52)
+		(end 132.73 65.02)
+		(width 0.25)
+		(layer "B.Cu")
+		(net 1)
+	)
+	(segment
 		(start 131.182 55.092)
 		(end 131.182 57.912936)
@@
 	)
 	(segment
-		(start 133.2925 62.712)
-		(end 133.2925 66.5845)
+		(start 132.73 65.02)
+		(end 133.484 65.774)
+		(width 0.25)
+		(layer "B.Cu")
+		(net 1)
+	)
+	(segment
+		(start 133.484 65.774)
+		(end 133.484 66.776)
 		(width 0.25)
 		(layer "B.Cu")
@@
 	)
 	(segment
-		(start 115.21316 61.188)
-		(end 122.546 68.52084)
-		(width 0.5)
-		(layer "B.Cu")
-		(net 6)
-	)
-	(segment
-		(start 115.18 48.531)
-		(end 115.18 61.188)
+		(start 114.73 48.981)
+		(end 114.73 58.77)
 		(width 0.5)
 		(layer "B.Cu")
@@
 	)
 	(segment
-		(start 122.546 68.52084)
+		(start 122.546 66.586)
 		(end 122.546 80.238)
 		(width 0.5)
@@
 	)
 	(segment
-		(start 122.546 80.238)
-		(end 124.34 82.032)
+		(start 114.73 58.77)
+		(end 122.546 66.586)
 		(width 0.5)
 		(layer "B.Cu")
@@
 	(segment
 		(start 118.111 45.6)
-		(end 115.18 48.531)
+		(end 114.73 48.981)
 		(width 0.5)
 		(layer "B.Cu")
@@
 	)
 	(segment
-		(start 115.18 61.188)
-		(end 115.21316 61.188)
+		(start 122.546 80.238)
+		(end 124.34 82.032)
 		(width 0.5)
 		(layer "B.Cu")
@@
 	)
 	(segment
+		(start 127.23 76.895)
+		(end 130.373835 80.038835)
+		(width 0.2)
+		(layer "B.Cu")
+		(net 17)
+	)
+	(segment
+		(start 130.373835 83.925835)
+		(end 130.48 84.032)
+		(width 0.2)
+		(layer "B.Cu")
+		(net 17)
+	)
+	(segment
+		(start 128.48 59.77)
+		(end 127.23 61.02)
+		(width 0.2)
+		(layer "B.Cu")
+		(net 17)
+	)
+	(segment
+		(start 130.373835 80.038835)
+		(end 130.373835 83.925835)
+		(width 0.2)
+		(layer "B.Cu")
+		(net 17)
+	)
+	(segment
 		(start 116.466 84.032)
 		(end 129.15 84.032)
@@
 	)
 	(segment
+		(start 127.23 61.02)
+		(end 127.23 76.895)
+		(width 0.2)
+		(layer "B.Cu")
+		(net 17)
+	)
+	(segment
 		(start 129.15 84.032)
+		(end 130.48 84.032)
+		(width 0.25)
+		(layer "B.Cu")
+		(net 17)
+	)
+	(segment
+		(start 130.48 84.032)
 		(end 131.69 84.032)
 		(width 0.25)
@@
 	)
 	(segment
+		(start 134.23 58.02)
+		(end 132.48 59.77)
+		(width 0.2)
+		(layer "B.Cu")
+		(net 17)
+	)
+	(segment
 		(start 131.706 84.016)
 		(end 131.69 84.032)
@@
 	)
 	(segment
+		(start 134.23 56.076)
+		(end 134.23 58.02)
+		(width 0.2)
+		(layer "B.Cu")
+		(net 17)
+	)
+	(segment
+		(start 132.48 59.77)
+		(end 128.48 59.77)
+		(width 0.2)
+		(layer "B.Cu")
+		(net 17)
+	)
+	(segment
 		(start 134.23 84.016)
 		(end 131.706 84.016)
@@
 	)
 	(segment
-		(start 139.63 61.762)
-		(end 135.1675 61.762)
+		(start 148.962 61.95)
+		(end 148.2 62.712)
 		(width 0.25)
 		(layer "B.Cu")
@@
 	)
 	(segment
-		(start 148.962 61.95)
-		(end 148.2 62.712)
+		(start 134.355 61.762)
+		(end 130.724 61.762)
 		(width 0.25)
 		(layer "B.Cu")
@@
 	)
 	(segment
-		(start 135.1175 61.712)
-		(end 135.1675 61.762)
+		(start 134.355 61.762)
+		(end 139.63 61.762)
 		(width 0.25)
 		(layer "B.Cu")
@@
 	)
 	(segment
-		(start 130.674 61.712)
-		(end 135.1175 61.712)
-		(width 0.25)
+		(start 130.724 61.762)
+		(end 130.674 61.712)
+		(width 0.2)
 		(layer "B.Cu")
 		(net 21)
@@
 	)
 	(segment
-		(start 135.1675 63.662)
-		(end 135.484 63.9785)
+		(start 134.355 63.662)
+		(end 134.355 64.395)
 		(width 0.25)
 		(layer "B.Cu")
@@
 	)
 	(segment
-		(start 135.484 63.9785)
-		(end 135.484 66.776)
+		(start 134.355 64.395)
+		(end 135.484 65.524)
 		(width 0.25)
 		(layer "B.Cu")
@@
 	)
 	(segment
+		(start 135.484 65.524)
+		(end 135.484 66.776)
+		(width 0.25)
+		(layer "B.Cu")
+		(net 28)
+	)
+	(segment
+		(start 134.23 54.076)
+		(end 134.23 53.068431)
+		(width 0.2)
+		(layer "B.Cu")
+		(net 36)
+	)
+	(segment
+		(start 134.23 53.068431)
+		(end 131.695037 50.533468)
+		(width 0.2)
+		(layer "B.Cu")
+		(net 36)
+	)
+	(segment
