File: ioboard.kicad_sch (KiCad schematic)
At the start: 37 parts, among them U3 TL431DBZ

Commit message: asd
Parts:
- R14: value 10k -> DNP
- R15: value 5k6 -> DNP
- R2: value 3.3M -> 2.2M
Connections:
- net at R14.1, R15.2, RV2.2: now also U3.1 (REF); no longer U3.2 (REF)
- net at R13.1, R14.2, R5.2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: now also U3.2 (K); no longer U3.1 (K)
Changed lines of the file:
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@@
 			)
 		)
-		(property "Value" "3.3M"
+		(property "Value" "2.2M"
 			(at 257.81 132.842 0)
 			(effects
@@
 			)
 		)
-		(property "Value" "10k"
+		(property "Value" "DNP"
 			(at 68.072 101.6 0)
 			(effects
@@
 			)
 		)
-		(property "Value" "5k6"
+		(property "Value" "DNP"
 			(at 68.072 115.57 0)
 			(effects
