File: mainboard.kicad_pcb (KiCad board)
At the start: 2 copper layers, 108 x 48.3 mm, 75 parts, among them IC1 LM555N, IC2 LM13700N, IC3 TL074P, IC4 TL074P

Commit message: asd
Parts:
- R20: value 2k -> 2k TEMPCO
- T3: value (none) -> 2N3904
- T4, T5: value (none) -> 2N3906 matched
Changed lines of the file:
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@@
 			)
 		)
-		(property "Value" "2k"
+		(property "Value" "2k TEMPCO"
 			(at -2.54 2.286 90)
 			(unlocked yes)
@@
 		)
 		(property "Footprint" ""
-			(at 0 0 -90)
+			(at 0 0 90)
 			(layer "F.Fab")
 			(hide yes)
@@
 		)
 		(property "Datasheet" ""
-			(at 0 0 -90)
+			(at 0 0 90)
 			(layer "F.Fab")
 			(hide yes)
@@
 		)
 		(property "Description" ""
-			(at 0 0 -90)
+			(at 0 0 90)
 			(layer "F.Fab")
 			(hide yes)
@@
 			)
 		)
-		(property "Value" ""
+		(property "Value" "2N3904"
 			(at -2.54 4.572 0)
 			(unlocked yes)
@@
 			)
 		)
-		(property "Value" ""
+		(property "Value" "2N3906 matched"
 			(at -2.54 4.572 90)
 			(unlocked yes)
@@
 		)
 		(property "Footprint" ""
-			(at 0 0 -90)
+			(at 0 0 90)
 			(layer "F.Fab")
 			(hide yes)
@@
 		)
 		(property "Datasheet" ""
-			(at 0 0 -90)
+			(at 0 0 90)
 			(layer "F.Fab")
 			(hide yes)
@@
 		)
 		(property "Description" ""
-			(at 0 0 -90)
+			(at 0 0 90)
 			(layer "F.Fab")
 			(hide yes)
@@
 			)
 		)
-		(property "Value" ""
+		(property "Value" "2N3906 matched"
 			(at -2.54 4.572 90)
 			(unlocked yes)
